Commit message: Got it to spawn in gazebo

File: workspace/src/six_dof_arm/urdf/kr120r2500pro.xacro (robot description, xacro)
@@ -2,5 +2,5 @@
 <!--Generates a urdf from the macro in kr120r2500pro_macro.xacro -->
 <robot name="kuka_kr120r2500pro" xmlns:xacro="http://wiki.ros.org/xacro">
-    <xacro:include filename="$(find kuka)/urdf/kr120r2500pro_macro.xacro" />
+    <xacro:include filename="$(find six_dof_arm)/urdf/kr120r2500pro_macro.xacro" />
     <xacro:kuka_kr120r2500pro prefix=""/>
 </robot>

File: workspace/src/six_dof_arm/urdf/kr120r2500pro_macro.xacro (robot description, xacro)
@@ -13,11 +13,11 @@
         <origin xyz="0 0 0" rpy="0 0 0"/>
         <geometry>
-          <mesh filename="package://kuka/meshes/kr120r2500pro/visual/base_link.dae" />
-        </geometry>
-      </visual>
-      <collision>
-        <origin xyz="0 0 0" rpy="0 0 0"/>
-        <geometry>
-          <mesh filename="package://kuka/meshes/kr120r2500pro/collision/base_link.stl" />
+          <mesh filename="package://six_dof_arm/meshes/kr120r2500pro/visual/base_link.dae" />
+        </geometry>
+      </visual>
+      <collision>
+        <origin xyz="0 0 0" rpy="0 0 0"/>
+        <geometry>
+          <mesh filename="package://six_dof_arm/meshes/kr120r2500pro/collision/base_link.stl" />
         </geometry>
       </collision>
@@ -33,11 +33,11 @@
         <origin xyz="0 0 0" rpy="0 0 0"/>
         <geometry>
-          <mesh filename="package://kuka/meshes/kr120r2500pro/visual/link_1.dae" />
-        </geometry>
-      </visual>
-      <collision>
-        <origin xyz="0 0 0" rpy="0 0 0"/>
-        <geometry>
-          <mesh filename="package://kuka/meshes/kr120r2500pro/collision/link_1.stl" />
+          <mesh filename="package://six_dof_arm/meshes/kr120r2500pro/visual/link_1.dae" />
+        </geometry>
+      </visual>
+      <collision>
+        <origin xyz="0 0 0" rpy="0 0 0"/>
+        <geometry>
+          <mesh filename="package://six_dof_arm/meshes/kr120r2500pro/collision/link_1.stl" />
         </geometry>
       </collision>
@@ -53,11 +53,11 @@
         <origin xyz="0 0 0" rpy="0 0 0"/>
         <geometry>
-          <mesh filename="package://kuka/meshes/kr120r2500pro/visual/link_2.dae"/>
-        </geometry>
-      </visual>
-      <collision>
-        <origin xyz="0 0 0" rpy="0 0 0"/>
-        <geometry>
-          <mesh filename="package://kuka/meshes/kr120r2500pro/collision/link_2.stl" />
+          <mesh filename="package://six_dof_arm/meshes/kr120r2500pro/visual/link_2.dae"/>
+        </geometry>
+      </visual>
+      <collision>
+        <origin xyz="0 0 0" rpy="0 0 0"/>
+        <geometry>
+          <mesh filename="package://six_dof_arm/meshes/kr120r2500pro/collision/link_2.stl" />
         </geometry>
       </collision>
@@ -73,11 +73,11 @@
         <origin xyz="0 0 0" rpy="0 0 0"/>
         <geometry>
-          <mesh filename="package://kuka/meshes/kr120r2500pro/visual/link_3.dae" />
-        </geometry>
-      </visual>
-      <collision>
-        <origin xyz="0 0 0" rpy="0 0 0"/>
-        <geometry>
-          <mesh filename="package://kuka/meshes/kr120r2500pro/collision/link_3.stl" />
+          <mesh filename="package://six_dof_arm/meshes/kr120r2500pro/visual/link_3.dae" />
+        </geometry>
+      </visual>
+      <collision>
+        <origin xyz="0 0 0" rpy="0 0 0"/>
+        <geometry>
+          <mesh filename="package://six_dof_arm/meshes/kr120r2500pro/collision/link_3.stl" />
         </geometry>
       </collision>
@@ -93,11 +93,11 @@
         <origin xyz="0 0 0" rpy="0 0 0"/>
         <geometry>
-          <mesh filename="package://kuka/meshes/kr120r2500pro/visual/link_4.dae" />
-        </geometry>
-      </visual>
-      <collision>
-        <origin xyz="0 0 0" rpy="0 0 0"/>
-        <geometry>
-          <mesh filename="package://kuka/meshes/kr120r2500pro/collision/link_4.stl" />
+          <mesh filename="package://six_dof_arm/meshes/kr120r2500pro/visual/link_4.dae" />
+        </geometry>
+      </visual>
+      <collision>
+        <origin xyz="0 0 0" rpy="0 0 0"/>
+        <geometry>
+          <mesh filename="package://six_dof_arm/meshes/kr120r2500pro/collision/link_4.stl" />
         </geometry>
       </collision>
@@ -113,11 +113,11 @@
         <origin xyz="0 0 0" rpy="0 0 0"/>
         <geometry>
-          <mesh filename="package://kuka/meshes/kr120r2500pro/visual/link_5.dae" />
-        </geometry>
-      </visual>
-      <collision>
-        <origin xyz="0 0 0" rpy="0 0 0"/>
-        <geometry>
-          <mesh filename="package://kuka/meshes/kr120r2500pro/collision/link_5.stl" />
+          <mesh filename="package://six_dof_arm/meshes/kr120r2500pro/visual/link_5.dae" />
+        </geometry>
+      </visual>
+      <collision>
+        <origin xyz="0 0 0" rpy="0 0 0"/>
+        <geometry>
+          <mesh filename="package://six_dof_arm/meshes/kr120r2500pro/collision/link_5.stl" />
         </geometry>
       </collision>
@@ -133,11 +133,11 @@
         <origin xyz="0 0 0" rpy="0 0 0"/>
         <geometry>
-          <mesh filename="package://kuka/meshes/kr120r2500pro/visual/link_6.dae" />
-        </geometry>
-      </visual>
-      <collision>
-        <origin xyz="0 0 0" rpy="0 0 0"/>
-        <geometry>
-          <mesh filename="package://kuka/meshes/kr120r2500pro/collision/link_6.stl" />
+          <mesh filename="package://six_dof_arm/meshes/kr120r2500pro/visual/link_6.dae" />
+        </geometry>
+      </visual>
+      <collision>
+        <origin xyz="0 0 0" rpy="0 0 0"/>
+        <geometry>
+          <mesh filename="package://six_dof_arm/meshes/kr120r2500pro/collision/link_6.stl" />
         </geometry>
       </collision>
@@ -217,5 +217,5 @@
     </joint>
     <!-- END JOINTS -->
-    <!-- ROS base_link to KUKA $ROBROOT coordinate system transform -->
+    <!-- ROS base_link to six_dof_arm $ROBROOT coordinate system transform -->
     <link name="${prefix}base" />
     <joint name="${prefix}base_link-base" type="fixed">
@@ -224,5 +224,5 @@
       <child link="${prefix}base"/>
     </joint>
-    <!-- This frame corresponds to the $TOOL coordinate system in KUKA KRC controllers -->
+    <!-- This frame corresponds to the $TOOL coordinate system in six_dof_arm KRC controllers -->
     <link name="${prefix}tool0" />
     <joint name="${prefix}flange-tool0" type="fixed">
@@ -231,73 +231,4 @@
       <origin xyz="0 0 0" rpy="0 ${radians(90)} 0"/>
     </joint>
-    <gazebo>
-        <!-- <plugin filename="libgz_ros2_control-system.so" name="gz_ros2_control::GazeboSimROS2ControlPlugin">
-          <parameters>$(find kuka)/config/controllers.yaml</parameters>
-        </plugin> -->
-        <plugin filename="/opt/ros/jazzy/lib/libgz_ros2_control-system.so" name="gz_ros2_control::GazeboSimROS2ControlPlugin">
-          <parameters>$(find kuka_moveit)/config/ros2_controllers.yaml</parameters>
-          <!-- <robot_param_node>robot_state_publisher</robot_param_node> -->
-        </plugin>
-        <plugin filename="gz-sim-joint-state-publisher-system"
-          name="gz::sim::systems::JointStatePublisher">
-          <topic>joint_states</topic> <!--from <ros><remapping> -->
-          <joint_name>joint_a1</joint_name>
-          <joint_name>joint_a2</joint_name>
-          <joint_name>joint_a3</joint_name>
-          <joint_name>joint_a4</joint_name>
-          <joint_name>joint_a5</joint_name>
-          <joint_name>joint_a6</joint_name>
-        </plugin>
-        <plugin
-          filename="gz-sim-joint-trajectory-controller-system"
-          name="gz::sim::systems::JointTrajectoryController">
-          <topic>/Arm_controller/joint_trajectory</topic>
-          <joint_name>joint_a1</joint_name>
-          <joint_name>joint_a2</joint_name>
-          <joint_name>joint_a3</joint_name>
-          <joint_name>joint_a4</joint_name>
-          <joint_name>joint_a5</joint_name>
-          <joint_name>joint_a6</joint_name>
-        </plugin>
-    </gazebo>
-    <ros2_control name="GazeboSystem" type="system">
-      <hardware>
-        <plugin>gz_ros2_control/GazeboSimSystem</plugin>
-      </hardware>
-  <!-- <ros2_control name="MockHardwareSystem" type="system">
-    <hardware>
-      <plugin>mock_components/GenericSystem</plugin>
-    </hardware> -->
-      <joint name="joint_a1">
-        <command_interface name="position"/>
-        <state_interface name="velocity"/>
-        <state_interface name="position"/>
-      </joint>
-      <joint name="joint_a2">
-        <command_interface name="position"/>
-        <state_interface name="velocity"/>
-        <state_interface name="position"/>
-      </joint>
-      <joint name="joint_a3">
-        <command_interface name="position"/>
-        <state_interface name="velocity"/>
-        <state_interface name="position"/>
-      </joint>
-      <joint name="joint_a4">
-        <command_interface name="position"/>
-        <state_interface name="velocity"/>
-        <state_interface name="position"/>
-      </joint>
-      <joint name="joint_a5">
-        <command_interface name="position"/>
-        <state_interface name="velocity"/>
-        <state_interface name="position"/>
-      </joint>
-      <joint name="joint_a6">
-        <command_interface name="position"/>
-        <state_interface name="velocity"/>
-        <state_interface name="position"/>
-      </joint>
-  </ros2_control>
   </xacro:macro>
 </robot>
