Commit message: The controllers are working too now

File: workspace/src/six_dof_arm/urdf/kr120r2500pro_macro.xacro (robot description, xacro)
@@ -231,4 +231,56 @@
       <origin xyz="0 0 0" rpy="0 ${radians(90)} 0"/>
     </joint>
+    <ros2_control name="GazeboSimSystem" type="system">
+      <hardware>
+        <plugin>gazebo_ros2_control/GazeboSystem</plugin>
+      </hardware>
+      <joint name="joint_a1">
+        <command_interface name="position"/>
+        <state_interface name="position">
+          <param name="initial_value">0.0</param>
+        </state_interface>
+        <state_interface name="velocity"/>
+      </joint>
+      <joint name="joint_a2">
+        <command_interface name="position"/>
+        <state_interface name="position">
+          <param name="initial_value">0.0</param>
+        </state_interface>
+        <state_interface name="velocity"/>
+      </joint>
+      <joint name="joint_a3">
+        <command_interface name="position"/>
+        <state_interface name="position">
+          <param name="initial_value">0.0</param>
+        </state_interface>
+        <state_interface name="velocity"/>
+      </joint>
+      <joint name="joint_a4">
+        <command_interface name="position"/>
+        <state_interface name="position">
+          <param name="initial_value">0.0</param>
+        </state_interface>
+        <state_interface name="velocity"/>
+      </joint>
+      <joint name="joint_a5">
+        <command_interface name="position"/>
+        <state_interface name="position">
+          <param name="initial_value">0.0</param>
+        </state_interface>
+        <state_interface name="velocity"/>
+      </joint>
+      <joint name="joint_a6">
+        <command_interface name="position"/>
+        <state_interface name="position">
+          <param name="initial_value">0.0</param>
+        </state_interface>
+        <state_interface name="velocity"/>
+      </joint>
+    </ros2_control>
+    <gazebo>
+      <plugin name="gazebo_ros2_control" filename="libgazebo_ros2_control.so">
+       <parameters>$(find six_dof_arm)/config/six_dof_arm_controllers.yaml</parameters>
+      </plugin>
+    </gazebo>
   </xacro:macro>
 </robot>

Commit message: Managed to get the PID working

File: workspace/src/six_dof_arm/urdf/kr120r2500pro_macro.xacro (robot description, xacro)
@@ -7,5 +7,5 @@
       <inertial>
         <origin xyz="0 0 0" rpy="0 0 0"/>
-        <mass value="2"/>
+        <mass value="80"/>
         <inertia ixx="0.01" ixy="0" ixz="0" iyy="0.01" iyz="0" izz="0.01" />
       </inertial>
@@ -27,5 +27,5 @@
       <inertial>
         <origin xyz="0 0 0" rpy="0 0 0"/>
-        <mass value="2"/>
+        <mass value="80"/>
         <inertia ixx="0.01" ixy="0" ixz="0" iyy="0.01" iyz="0" izz="0.01" />
       </inertial>
@@ -47,5 +47,5 @@
       <inertial>
         <origin xyz="0 0 0" rpy="0 0 0"/>
-        <mass value="2"/>
+        <mass value="80"/>
         <inertia ixx="0.01" ixy="0" ixz="0" iyy="0.01" iyz="0" izz="0.01" />
       </inertial>
@@ -67,5 +67,5 @@
       <inertial>
         <origin xyz="0 0 0" rpy="0 0 0"/>
-        <mass value="2"/>
+        <mass value="80"/>
         <inertia ixx="0.01" ixy="0" ixz="0" iyy="0.01" iyz="0" izz="0.01" />
       </inertial>
@@ -87,5 +87,5 @@
       <inertial>
         <origin xyz="0 0 0" rpy="0 0 0"/>
-        <mass value="2"/>
+        <mass value="80"/>
         <inertia ixx="0.01" ixy="0" ixz="0" iyy="0.01" iyz="0" izz="0.01" />
       </inertial>
@@ -107,5 +107,5 @@
       <inertial>
         <origin xyz="0 0 0" rpy="0 0 0"/>
-        <mass value="2"/>
+        <mass value="80"/>
         <inertia ixx="0.01" ixy="0" ixz="0" iyy="0.01" iyz="0" izz="0.01" />
       </inertial>
@@ -127,5 +127,5 @@
       <inertial>
         <origin xyz="0 0 0" rpy="0 0 0"/>
-        <mass value="2"/>
+        <mass value="80"/>
         <inertia ixx="0.01" ixy="0" ixz="0" iyy="0.01" iyz="0" izz="0.01" />
       </inertial>
@@ -236,44 +236,62 @@
       </hardware>
       <joint name="joint_a1">
-        <command_interface name="position"/>
-        <state_interface name="position">
-          <param name="initial_value">0.0</param>
-        </state_interface>
-        <state_interface name="velocity"/>
+        <!--<command_interface name="position"/>-->
+        <command_interface name="position_pid"/>
+        <command_interface name="effort"/>
+        <state_interface name="position">
+          <param name="initial_value">0.0</param>
+        </state_interface>
+        <state_interface name="velocity"/>
+        <state_interface name="effort"/>
       </joint>
       <joint name="joint_a2">
-        <command_interface name="position"/>
-        <state_interface name="position">
-          <param name="initial_value">0.0</param>
-        </state_interface>
-        <state_interface name="velocity"/>
+        <!--<command_interface name="position"/>-->
+        <command_interface name="position_pid"/>
+        <command_interface name="effort"/>
+        <state_interface name="position">
+          <param name="initial_value">0.0</param>
+        </state_interface>
+        <state_interface name="velocity"/>
+        <state_interface name="effort"/>
       </joint>
       <joint name="joint_a3">
-        <command_interface name="position"/>
-        <state_interface name="position">
-          <param name="initial_value">0.0</param>
-        </state_interface>
-        <state_interface name="velocity"/>
+        <!--<command_interface name="position"/>-->
+        <command_interface name="position_pid"/>
+        <command_interface name="effort"/>
+        <state_interface name="position">
+          <param name="initial_value">0.0</param>
+        </state_interface>
+        <state_interface name="velocity"/>
+        <state_interface name="effort"/>
       </joint>
       <joint name="joint_a4">
-        <command_interface name="position"/>
-        <state_interface name="position">
-          <param name="initial_value">0.0</param>
-        </state_interface>
-        <state_interface name="velocity"/>
+        <!--<command_interface name="position"/>-->
+        <command_interface name="position_pid"/>
+        <command_interface name="effort"/>
+        <state_interface name="position">
+          <param name="initial_value">0.0</param>
+        </state_interface>
+        <state_interface name="velocity"/>
+        <state_interface name="effort"/>
       </joint>
       <joint name="joint_a5">
-        <command_interface name="position"/>
-        <state_interface name="position">
-          <param name="initial_value">0.0</param>
-        </state_interface>
-        <state_interface name="velocity"/>
+        <!--<command_interface name="position"/>-->
+        <command_interface name="position_pid"/>
+        <command_interface name="effort"/>
+        <state_interface name="position">
+          <param name="initial_value">0.0</param>
+        </state_interface>
+        <state_interface name="velocity"/>
+        <state_interface name="effort"/>
       </joint>
       <joint name="joint_a6">
-        <command_interface name="position"/>
-        <state_interface name="position">
-          <param name="initial_value">0.0</param>
-        </state_interface>
-        <state_interface name="velocity"/>
+        <!--<command_interface name="position"/>-->
+        <command_interface name="position_pid"/>
+        <command_interface name="effort"/>
+        <state_interface name="position">
+          <param name="initial_value">0.0</param>
+        </state_interface>
+        <state_interface name="velocity"/>
+        <state_interface name="effort"/>
       </joint>
     </ros2_control>

Commit message: Working froce torque sensors

File: workspace/src/six_dof_arm/urdf/kr120r2500pro_macro.xacro (robot description, xacro)
@@ -7,5 +7,5 @@
       <inertial>
         <origin xyz="0 0 0" rpy="0 0 0"/>
-        <mass value="80"/>
+        <mass value="2"/>
         <inertia ixx="0.01" ixy="0" ixz="0" iyy="0.01" iyz="0" izz="0.01" />
       </inertial>
@@ -27,5 +27,5 @@
       <inertial>
         <origin xyz="0 0 0" rpy="0 0 0"/>
-        <mass value="80"/>
+        <mass value="2"/>
         <inertia ixx="0.01" ixy="0" ixz="0" iyy="0.01" iyz="0" izz="0.01" />
       </inertial>
@@ -47,5 +47,5 @@
       <inertial>
         <origin xyz="0 0 0" rpy="0 0 0"/>
-        <mass value="80"/>
+        <mass value="2"/>
         <inertia ixx="0.01" ixy="0" ixz="0" iyy="0.01" iyz="0" izz="0.01" />
       </inertial>
@@ -67,5 +67,5 @@
       <inertial>
         <origin xyz="0 0 0" rpy="0 0 0"/>
-        <mass value="80"/>
+        <mass value="2"/>
         <inertia ixx="0.01" ixy="0" ixz="0" iyy="0.01" iyz="0" izz="0.01" />
       </inertial>
@@ -87,5 +87,5 @@
       <inertial>
         <origin xyz="0 0 0" rpy="0 0 0"/>
-        <mass value="80"/>
+        <mass value="2"/>
         <inertia ixx="0.01" ixy="0" ixz="0" iyy="0.01" iyz="0" izz="0.01" />
       </inertial>
@@ -107,5 +107,5 @@
       <inertial>
         <origin xyz="0 0 0" rpy="0 0 0"/>
-        <mass value="80"/>
+        <mass value="2"/>
         <inertia ixx="0.01" ixy="0" ixz="0" iyy="0.01" iyz="0" izz="0.01" />
       </inertial>
@@ -127,5 +127,5 @@
       <inertial>
         <origin xyz="0 0 0" rpy="0 0 0"/>
-        <mass value="80"/>
+        <mass value="2"/>
         <inertia ixx="0.01" ixy="0" ixz="0" iyy="0.01" iyz="0" izz="0.01" />
       </inertial>
@@ -301,4 +301,70 @@
       </plugin>
     </gazebo>
+    <gazebo reference="joint_a1">
+      <sensor name="joint_a1_force_torque" type="force_torque">
+        <always_on>true</always_on>
+        <update_rate>20.0</update_rate>
+        <visualize>true</visualize>
+        <force_torque>
+          <frame>sensor</frame>
+          <measure_direction>child_to_parent</measure_direction>
+        </force_torque>
+      </sensor>
+    </gazebo>
+    <gazebo reference="joint_a2">
+      <sensor name="joint_a2_force_torque" type="force_torque">
+        <always_on>true</always_on>
+        <update_rate>20.0</update_rate>
+        <visualize>true</visualize>
+        <force_torque>
+          <frame>sensor</frame>
+          <measure_direction>child_to_parent</measure_direction>
+        </force_torque>
+      </sensor>
+    </gazebo>
+    <gazebo reference="joint_a3">
+      <sensor name="joint_a3_force_torque" type="force_torque">
+        <always_on>true</always_on>
+        <update_rate>20.0</update_rate>
+        <visualize>true</visualize>
+        <force_torque>
+          <frame>sensor</frame>
+          <measure_direction>child_to_parent</measure_direction>
+        </force_torque>
+      </sensor>
+    </gazebo>
+    <gazebo reference="joint_a4">
+      <sensor name="joint_a4_force_torque" type="force_torque">
+        <always_on>true</always_on>
+        <update_rate>20.0</update_rate>
+        <visualize>true</visualize>
+        <force_torque>
+          <frame>sensor</frame>
+          <measure_direction>child_to_parent</measure_direction>
+        </force_torque>
+      </sensor>
+    </gazebo>
+    <gazebo reference="joint_a5">
+      <sensor name="joint_a5_force_torque" type="force_torque">
+        <always_on>true</always_on>
+        <update_rate>20.0</update_rate>
+        <visualize>true</visualize>
+        <force_torque>
+          <frame>sensor</frame>
+          <measure_direction>child_to_parent</measure_direction>
+        </force_torque>
+      </sensor>
+    </gazebo>
+    <gazebo reference="joint_a6">
+      <sensor name="joint_a6_force_torque" type="force_torque">
+        <always_on>true</always_on>
+        <update_rate>20.0</update_rate>
+        <visualize>true</visualize>
+        <force_torque>
+          <frame>sensor</frame>
+          <measure_direction>child_to_parent</measure_direction>
+        </force_torque>
+      </sensor>
+    </gazebo>
   </xacro:macro>
 </robot>

Commit message: dynamics basically done

File: workspace/src/six_dof_arm/urdf/kr120r2500pro_macro.xacro (robot description, xacro)
@@ -4,4 +4,5 @@
     <!-- LINKS -->
     <!-- base link -->
+    <link name="world"></link>
     <link name="${prefix}base_link">
       <inertial>
@@ -27,5 +28,5 @@
       <inertial>
         <origin xyz="0 0 0" rpy="0 0 0"/>
-        <mass value="2"/>
+        <mass value="209"/>
         <inertia ixx="0.01" ixy="0" ixz="0" iyy="0.01" iyz="0" izz="0.01" />
       </inertial>
@@ -47,5 +48,5 @@
       <inertial>
         <origin xyz="0 0 0" rpy="0 0 0"/>
-        <mass value="2"/>
+        <mass value="316"/>
         <inertia ixx="0.01" ixy="0" ixz="0" iyy="0.01" iyz="0" izz="0.01" />
       </inertial>
@@ -67,5 +68,5 @@
       <inertial>
         <origin xyz="0 0 0" rpy="0 0 0"/>
-        <mass value="2"/>
+        <mass value="79.9"/>
         <inertia ixx="0.01" ixy="0" ixz="0" iyy="0.01" iyz="0" izz="0.01" />
       </inertial>
@@ -87,5 +88,5 @@
       <inertial>
         <origin xyz="0 0 0" rpy="0 0 0"/>
-        <mass value="2"/>
+        <mass value="27.3"/>
         <inertia ixx="0.01" ixy="0" ixz="0" iyy="0.01" iyz="0" izz="0.01" />
       </inertial>
@@ -107,5 +108,5 @@
       <inertial>
         <origin xyz="0 0 0" rpy="0 0 0"/>
-        <mass value="2"/>
+        <mass value="50"/>
         <inertia ixx="0.01" ixy="0" ixz="0" iyy="0.01" iyz="0" izz="0.01" />
       </inertial>
@@ -146,4 +147,9 @@
     <link name="${prefix}flange" />
     <!-- END LINKS -->
+    <joint name="${prefix}world_joint" type="fixed">
+      <origin xyz="1.5 1.0 0" rpy="0 0 0"/>
+      <parent link="world"/>
+      <child link="${prefix}base_link"/>
+    </joint>
     <!-- JOINTS -->
     <!-- joint 1 (A1) -->
@@ -344,5 +350,5 @@
       <sensor name="joint_a1_force_torque" type="force_torque">
         <always_on>true</always_on>
-        <update_rate>20.0</update_rate>
+        <update_rate>100.0</update_rate>
         <visualize>true</visualize>
         <force_torque>
@@ -355,5 +361,5 @@
       <sensor name="joint_a2_force_torque" type="force_torque">
         <always_on>true</always_on>
-        <update_rate>20.0</update_rate>
+        <update_rate>100.0</update_rate>
         <visualize>true</visualize>
         <force_torque>
@@ -366,5 +372,5 @@
       <sensor name="joint_a3_force_torque" type="force_torque">
         <always_on>true</always_on>
-        <update_rate>20.0</update_rate>
+        <update_rate>100.0</update_rate>
         <visualize>true</visualize>
         <force_torque>
@@ -377,5 +383,5 @@
       <sensor name="joint_a4_force_torque" type="force_torque">
         <always_on>true</always_on>
-        <update_rate>20.0</update_rate>
+        <update_rate>100.0</update_rate>
         <visualize>true</visualize>
         <force_torque>
@@ -388,5 +394,5 @@
       <sensor name="joint_a5_force_torque" type="force_torque">
         <always_on>true</always_on>
-        <update_rate>20.0</update_rate>
+        <update_rate>100.0</update_rate>
         <visualize>true</visualize>
         <force_torque>
@@ -399,5 +405,5 @@
       <sensor name="joint_a6_force_torque" type="force_torque">
         <always_on>true</always_on>
-        <update_rate>20.0</update_rate>
+        <update_rate>100.0</update_rate>
         <visualize>true</visualize>
         <force_torque>
