Commit message: Working leg1

File: workspace/src/gantry2/urdf/gantry.xacro (robot description, xacro)
@@ -1,40 +1,19 @@
 <?xml version="1.0"?>
 <robot xmlns:xacro="http://www.ros.org/wiki/xacro" name="rectangular_gantry">
-  <!-- Params -->
-  <xacro:property name="length_x" value="1.5" />    <!-- travel along X (m) -->
-  <xacro:property name="length_y" value="1.0" />    <!-- travel along Y (m) -->
-  <xacro:property name="height" value="0.2" />    <!-- rail height (m) -->
-  <xacro:property name="rail_w" value="0.06" />   <!-- rail width (m) -->
-  <xacro:property name="base_th" value="0.08" />   <!-- base thickness (m) -->
-  <xacro:property name="car_w" value="0.18" />   <!-- carriage width (m) -->
-  <xacro:property name="car_h" value="0.08" />   <!-- carriage height (m) -->
-  <xacro:property name="mass_base" value="10.0" />
-  <xacro:property name="mass_gantry" value="6.0" />
-  <xacro:property name="mass_carriage" value="1.0" />
-  <!-- Inertial helper macro (simple box inertia approx) -->
-  <xacro:macro name="box_inertial" params="nx ny nz mass">
-    <inertial>
-      <origin xyz="0 0 0" rpy="0 0 0" />
-      <mass value="${mass}" />
-      <!-- very rough inertia (diagonal) -->
-      <inertia ixx="${(1.0/12.0)*mass*(ny*ny + nz*nz)}"
-        ixy="0" ixz="0"
-        iyy="${(1.0/12.0)*mass*(nx*nx + nz*nz)}"
-        iyz="0"
-        izz="${(1.0/12.0)*mass*(nx*nx + ny*ny)}" />
-    </inertial>
-  </xacro:macro>
+  <xacro:property name="length_leg" value="1" />    <!-- travel along X (m) -->
+  <xacro:property name="thickness_leg" value="0.2" />    <!-- travel along X (m) -->
+  <xacro:property name="width_leg" value="0.2" />    <!-- travel along X (m) -->
+  <xacro:property name="mass_leg" value="1" />    <!-- travel along X (m) -->
   <link name="map" />
-  <joint name="map_to_base" type="fixed">
+  <joint name="map_to_leg1" type="fixed">
     <parent link="map" />
-    <child link="base_link" />
+    <child link="leg1" />
     <origin xyz="0 0 0" rpy="0 0 0" />
   </joint>
-  <!-- Base link -->
-  <link name="base_link">
+  <link name="leg1">
     <visual>
-      <origin xyz="0 0 ${-base_th/2}" rpy="0 0 0" />
+      <origin xyz="0 0 0" rpy="0 -${pi/2} 0" />
       <geometry>
-        <box size="${length_x} ${length_y} ${base_th}" />
+        <box size="${length_leg} ${width_leg} ${thickness_leg}" />
       </geometry>
       <material name="gray">
@@ -43,132 +22,14 @@
     </visual>
     <collision>
-      <origin xyz="0 0 ${-base_th/2}" rpy="0 0 0" />
+      <origin xyz="0 0 0" rpy="0 -${pi/2} 0" />
       <geometry>
-        <box size="${length_x} ${length_y} ${base_th}" />
+        <box size="${length_leg} ${width_leg} ${thickness_leg}" />
       </geometry>
     </collision>
     <inertial>
-      <origin xyz="0 0 0" rpy="0 0 0" />
-      <mass value="${mass_base}" />
+      <origin xyz="0 0 0" rpy="0 -${pi/2} 0" />
+      <mass value="${mass_leg}" />
       <inertia ixx="1.0" ixy="0" ixz="0" iyy="1.0" iyz="0" izz="1.0" />
     </inertial>
   </link>
-  <!-- Gantry (moves in Y) -->
-  <link name="gantry_y_link">
-    <visual>
-      <!-- two parallel X-rails (left & right) -->
-      <origin xyz="0 ${length_y/2 - rail_w/2} ${height/2}" rpy="0 0 0" />
-      <geometry>
-        <box size="${length_x} ${rail_w} ${height}" />
-      </geometry>
-      <material name="dark">
-        <color rgba="0.3 0.3 0.3 1.0" />
-      </material>
-    </visual>
-    <visual>
-      <origin xyz="0 ${- (length_y/2 - rail_w/2)} ${height/2}" rpy="0 0 0" />
-      <geometry>
-        <box size="${length_x} ${rail_w} ${height}" />
-      </geometry>
-      <material name="dark" />
-    </visual>
-    <collision>
-      <origin xyz="0 ${length_y/2 - rail_w/2} ${height/2}" rpy="0 0 0" />
-      <geometry>
-        <box size="${length_x} ${rail_w} ${height}" />
-      </geometry>
-    </collision>
-    <collision>
-      <origin xyz="0 ${- (length_y/2 - rail_w/2)} ${height/2}" rpy="0 0 0" />
-      <geometry>
-        <box size="${length_x} ${rail_w} ${height}" />
-      </geometry>
-    </collision>
-    <inertial>
-      <origin xyz="0 0 ${height/2}" rpy="0 0 0" />
-      <mass value="${mass_gantry}" />
-      <inertia ixx="0.5" ixy="0" ixz="0" iyy="0.5" iyz="0" izz="0.5" />
-    </inertial>
-  </link>
-  <!-- Joint: gantry sliding along Y relative to base -->
-  <joint name="gantry_y_prismatic" type="prismatic">
-    <parent link="base_link" />
-    <child link="gantry_y_link" />
-    <origin xyz="0 0 0" rpy="0 0 0" />
-    <axis xyz="0 1 0" />
-    <limit lower="${-length_y/2}" upper="${length_y/2}" effort="1000" velocity="0.5" />
-  </joint>
-  <!-- Carriage (moves along X, attached to gantry_y_link) -->
-  <link name="carriage_link">
-    <visual>
-      <origin xyz="0 0 ${car_h/2 + height/2}" rpy="0 0 0" />
-      <geometry>
-        <box size="${car_w} ${rail_w*2 + 0.02} ${car_h}" />
-      </geometry>
-      <material name="blue">
-        <color rgba="0.2 0.4 0.8 1.0" />
-      </material>
-    </visual>
-    <collision>
-      <origin xyz="0 0 ${car_h/2 + height/2}" rpy="0 0 0" />
-      <geometry>
-        <box size="${car_w} ${rail_w*2 + 0.02} ${car_h}" />
-      </geometry>
-    </collision>
-    <inertial>
-      <origin xyz="0 0 ${car_h/2 + height/2}" rpy="0 0 0" />
-      <mass value="${mass_carriage}" />
-      <inertia ixx="0.01" ixy="0" ixz="0" iyy="0.01" iyz="0" izz="0.01" />
-    </inertial>
-  </link>
-  <!-- Joint: carriage sliding along X on top of gantry -->
-  <joint name="carriage_x_prismatic" type="prismatic">
-    <parent link="gantry_y_link" />
-    <child link="carriage_link" />
-    <!-- place carriage initially centered -->
-    <origin xyz="0 0 0" rpy="0 0 0" />
-    <axis xyz="1 0 0" />
-    <limit lower="${-length_x/2}" upper="${length_x/2}" effort="500" velocity="0.6" />
-  </joint>
-  <!-- Optional tool mount on carriage -->
-  <link name="tool_mount">
-    <visual>
-      <origin xyz="0 0 ${-car_h/2}" rpy="0 0 0" />
-      <geometry>
-        <cylinder length="0.05" radius="0.02" />
-      </geometry>
-      <material name="red">
-        <color rgba="0.8 0.2 0.2 1.0" />
-      </material>
-    </visual>
-    <collision>
-      <origin xyz="0 0 ${-car_h/2}" rpy="0 0 0" />
-      <geometry>
-        <cylinder length="0.05" radius="0.02" />
-      </geometry>
-    </collision>
-    <inertial>
-      <origin xyz="0 0 0" rpy="0 0 0" />
-      <mass value="0.1" />
-      <inertia ixx="1e-4" ixy="0" ixz="0" iyy="1e-4" iyz="0" izz="1e-4" />
-    </inertial>
-  </link>
-  <joint name="carriage_tool_fixed" type="fixed">
-    <parent link="carriage_link" />
-    <child link="tool_mount" />
-    <origin xyz="0 0 ${-car_h/2}" rpy="0 0 0" />
-  </joint>
-  <!-- Gazebo-friendly transmission hints (optional) -->
-  <xacro:property name="controller_namespace" value="" />
-  <transmission name="gantry_y_trans">
-    <type>transmission_interface/SimpleTransmission</type>
-    <joint name="gantry_y_prismatic" />
-    <actuator name="gantry_y_motor" />
-  </transmission>
-  <transmission name="carriage_x_trans">
-    <type>transmission_interface/SimpleTransmission</type>
-    <joint name="carriage_x_prismatic" />
-    <actuator name="carriage_x_motor" />
-  </transmission>
-  <!-- End -->
 </robot>

Commit message: Added legs

File: workspace/src/gantry2/urdf/gantry.xacro (robot description, xacro)
@@ -1,35 +1,41 @@
 <?xml version="1.0"?>
 <robot xmlns:xacro="http://www.ros.org/wiki/xacro" name="rectangular_gantry">
-  <xacro:property name="length_leg" value="1" />    <!-- travel along X (m) -->
-  <xacro:property name="thickness_leg" value="0.2" />    <!-- travel along X (m) -->
-  <xacro:property name="width_leg" value="0.2" />    <!-- travel along X (m) -->
-  <xacro:property name="mass_leg" value="1" />    <!-- travel along X (m) -->
+  <xacro:property name="length_bar" value="1" />    <!-- travel along X (m) -->
+  <xacro:property name="thickness_bar" value="0.2" />    <!-- travel along X (m) -->
+  <xacro:property name="width_bar" value="0.2" />    <!-- travel along X (m) -->
+  <xacro:property name="mass_bar" value="1" />    <!-- travel along X (m) -->
+  <xacro:macro name="bar" params="name parent xyz rpy">
+    <link name="${name}">
+      <visual>
+        <origin xyz="0 0 0" rpy="0 0 0" />
+        <geometry>
+          <box size="${length_bar} ${width_bar} ${thickness_bar}" />
+        </geometry>
+        <material name="gray">
+          <color rgba="0.6 0.6 0.6 1.0" />
+        </material>
+      </visual>
+      <collision>
+        <origin xyz="0 0 0" rpy="0 0 0" />
+        <geometry>
+          <box size="${length_bar} ${width_bar} ${thickness_bar}" />
+        </geometry>
+      </collision>
+      <inertial>
+        <origin xyz="0 0 0" rpy="0 0 0" />
+        <mass value="${mass_bar}" />
+        <inertia ixx="1.0" ixy="0" ixz="0" iyy="1.0" iyz="0" izz="1.0" />
+      </inertial>
+    </link>
+    <joint name="${parent}_to_${name}" type="fixed">
+      <parent link="${parent}" />
+      <child link="${name}" />
+      <origin xyz="${xyz}" rpy="${rpy}" />
+    </joint>
+  </xacro:macro>
   <link name="map" />
-  <joint name="map_to_leg1" type="fixed">
-    <parent link="map" />
-    <child link="leg1" />
-    <origin xyz="0 0 0" rpy="0 0 0" />
-  </joint>
-  <link name="leg1">
-    <visual>
-      <origin xyz="0 0 0" rpy="0 -${pi/2} 0" />
-      <geometry>
-        <box size="${length_leg} ${width_leg} ${thickness_leg}" />
-      </geometry>
-      <material name="gray">
-        <color rgba="0.6 0.6 0.6 1.0" />
-      </material>
-    </visual>
-    <collision>
-      <origin xyz="0 0 0" rpy="0 -${pi/2} 0" />
-      <geometry>
-        <box size="${length_leg} ${width_leg} ${thickness_leg}" />
-      </geometry>
-    </collision>
-    <inertial>
-      <origin xyz="0 0 0" rpy="0 -${pi/2} 0" />
-      <mass value="${mass_leg}" />
-      <inertia ixx="1.0" ixy="0" ixz="0" iyy="1.0" iyz="0" izz="1.0" />
-    </inertial>
-  </link>
+  <xacro:bar name="bar1" parent="map" xyz="0 0 0" rpy="0 -${pi/2} 0" />
+  <xacro:bar name="bar2" parent="map" xyz="-${length_bar} 0 0" rpy="0 -${pi/2} 0" />
+  <xacro:bar name="bar3" parent="map" xyz="-${length_bar} -${length_bar} 0" rpy="0 -${pi/2} 0" />
+  <xacro:bar name="bar4" parent="map" xyz="0 -${length_bar} 0" rpy="0 -${pi/2} 0" />
 </robot>

Commit message: Thinner gantry

File: workspace/src/gantry2/urdf/gantry.xacro (robot description, xacro)
@@ -2,6 +2,6 @@
 <robot xmlns:xacro="http://www.ros.org/wiki/xacro" name="rectangular_gantry">
   <xacro:property name="length_bar" value="1" />    <!-- travel along X (m) -->
-  <xacro:property name="thickness_bar" value="0.2" />    <!-- travel along X (m) -->
-  <xacro:property name="width_bar" value="0.2" />    <!-- travel along X (m) -->
+  <xacro:property name="thickness_bar" value="0.02" />    <!-- travel along X (m) -->
+  <xacro:property name="width_bar" value="0.02" />    <!-- travel along X (m) -->
   <xacro:property name="mass_bar" value="1" />    <!-- travel along X (m) -->
   <xacro:macro name="bar" params="name parent xyz rpy">
@@ -51,3 +51,5 @@
     rpy="0 0 0" />
   <!-- This is from 3 and 4  -->
+  <xacro:bar name="xaxis" parent="map" xyz="0 -${length_bar/2} ${length_bar+width_bar}"
+    rpy="0 0 -${pi/2}" />
 </robot>

Commit message: Working layers

File: workspace/src/gantry2/urdf/gantry.xacro (robot description, xacro)
@@ -5,5 +5,6 @@
   <xacro:property name="width_bar" value="0.02" />    <!-- travel along X (m) -->
   <xacro:property name="mass_bar" value="1" />    <!-- travel along X (m) -->
-  <xacro:macro name="bar" params="name parent xyz rpy">
+  <!-- Macro for a bar -->
+  <xacro:macro name="bar" params="name">
     <link name="${name}">
       <visual>
@@ -28,28 +29,37 @@
       </inertial>
     </link>
-    <joint name="${parent}_to_${name}" type="fixed">
+  </xacro:macro>
+  <!-- Macro for a fixed joint -->
+  <xacro:macro name="fixed_joint" params="parent child xyz rpy">
+    <joint name="${parent}_to_${child}" type="fixed">
       <parent link="${parent}" />
-      <child link="${name}" />
+      <child link="${child}" />
       <origin xyz="${xyz}" rpy="${rpy}" />
     </joint>
   </xacro:macro>
+  <!-- Base link -->
   <link name="map" />
-  <xacro:bar name="leg1" parent="map" xyz="0 0 ${length_bar/2}" rpy="0 -${pi/2} 0" />
-  <xacro:bar name="leg2" parent="map" xyz="-${length_bar} 0 ${length_bar/2}" rpy="0 -${pi/2} 0" />
-  <xacro:bar name="layer1" parent="map" xyz="-${length_bar/2} 0 ${length_bar}"
+  <!-- Bars + joints -->
+  <xacro:bar name="leg1" />
+  <xacro:fixed_joint parent="map" child="leg1" xyz="0 0 ${length_bar/2}" rpy="0 -${pi/2} 0" />
+  <xacro:bar name="leg2" />
+  <xacro:fixed_joint parent="map" child="leg2" xyz="-${length_bar} 0 ${length_bar/2}"
+    rpy="0 -${pi/2} 0" />
+  <xacro:bar name="layer1" />
+  <xacro:fixed_joint parent="map" child="layer1" xyz="-${length_bar/2} 0 ${length_bar}" rpy="0 0 0" />
+  <xacro:bar name="layer2" />
+  <xacro:fixed_joint parent="map" child="layer2" xyz="-${length_bar} -${length_bar/2} ${length_bar}"
+    rpy="0 0 -${pi/2}" />
+  <xacro:bar name="leg3" />
+  <xacro:fixed_joint parent="map" child="leg3" xyz="-${length_bar} -${length_bar} ${length_bar/2}"
+    rpy="0 -${pi/2} 0" />
+  <xacro:bar name="layer3" />
+  <xacro:fixed_joint parent="map" child="layer3" xyz="0 -${length_bar/2} ${length_bar}"
+    rpy="0 0 -${pi/2}" />
+  <xacro:bar name="leg4" />
+  <xacro:fixed_joint parent="map" child="leg4" xyz="0 -${length_bar} ${length_bar/2}"
+    rpy="0 -${pi/2} 0" />
+  <xacro:bar name="layer4" />
+  <xacro:fixed_joint parent="map" child="layer4" xyz="-${length_bar/2} -${length_bar} ${length_bar}"
     rpy="0 0 0" />
-  <!-- This is from 1 and 2 -->
-  <xacro:bar name="layer2" parent="map" xyz="-${length_bar} -${length_bar/2} ${length_bar}"
-    rpy="0 0 -${pi/2}" />
-  <!-- This is from 2 and 3  -->
-  <xacro:bar name="leg3" parent="map" xyz="-${length_bar} -${length_bar} ${length_bar/2}"
-    rpy="0 -${pi/2} 0" />
-  <xacro:bar name="layer3" parent="map" xyz="0 -${length_bar/2} ${length_bar}"
-    rpy="0 0 -${pi/2}" />
-  <xacro:bar name="leg4" parent="map" xyz="0 -${length_bar} ${length_bar/2} " rpy="0 -${pi/2} 0" />
-  <xacro:bar name="layer4" parent="map" xyz="-${length_bar/2} -${length_bar} ${length_bar}"
-    rpy="0 0 0" />
-  <!-- This is from 3 and 4  -->
-  <xacro:bar name="xaxis" parent="map" xyz="0 -${length_bar/2} ${length_bar+width_bar}"
-    rpy="0 0 -${pi/2}" />
 </robot>

Commit message: Working one railing

File: workspace/src/gantry2/urdf/gantry.xacro (robot description, xacro)
@@ -38,4 +38,13 @@
     </joint>
   </xacro:macro>
+  <xacro:macro name="prismatic_joint" params="parent child xyz rpy axis lower upper">
+    <joint name="${parent}_to_${child}" type="prismatic">
+      <parent link="${parent}" />
+      <child link="${child}" />
+      <origin xyz="${xyz}" rpy="${rpy}" />
+      <axis xyz="${axis}" />
+      <limit lower="${lower}" upper="${upper}" effort="100" velocity="1.0" />
+    </joint>
+  </xacro:macro>
   <!-- Base link -->
   <link name="map" />
@@ -63,3 +72,9 @@
   <xacro:fixed_joint parent="map" child="layer4" xyz="-${length_bar/2} -${length_bar} ${length_bar}"
     rpy="0 0 0" />
+  <xacro:bar name="xaxis" />
+  <xacro:prismatic_joint parent="map" child="xaxis"
+    xyz="0 -${length_bar/2} ${length_bar}"
+    rpy="0 0 -${pi/2}"
+    axis="0 1 0"
+    lower="-${length_bar}" upper="0" />
 </robot>

Commit message: Was able to refactor for size

File: workspace/src/gantry2/urdf/gantry.xacro (robot description, xacro)
@@ -6,10 +6,10 @@
   <xacro:property name="mass_bar" value="1" />    <!-- travel along X (m) -->
   <!-- Macro for a bar -->
-  <xacro:macro name="bar" params="name">
+  <xacro:macro name="bar" params="name length width thickness">
     <link name="${name}">
       <visual>
         <origin xyz="0 0 0" rpy="0 0 0" />
         <geometry>
-          <box size="${length_bar} ${width_bar} ${thickness_bar}" />
+          <box size="${length} ${width} ${thickness}" />
         </geometry>
         <material name="gray">
@@ -20,5 +20,5 @@
         <origin xyz="0 0 0" rpy="0 0 0" />
         <geometry>
-          <box size="${length_bar} ${width_bar} ${thickness_bar}" />
+          <box size="${length} ${width} ${thickness}" />
         </geometry>
       </collision>
@@ -50,27 +50,27 @@
   <link name="map" />
   <!-- Bars + joints -->
-  <xacro:bar name="leg1" />
+  <xacro:bar name="leg1" length="${length_bar}" width="${width_bar}" thickness="${thickness_bar}" />
   <xacro:fixed_joint parent="map" child="leg1" xyz="0 0 ${length_bar/2}" rpy="0 -${pi/2} 0" />
-  <xacro:bar name="leg2" />
+  <xacro:bar name="leg2" length="${length_bar}" width="${width_bar}" thickness="${thickness_bar}" />
   <xacro:fixed_joint parent="map" child="leg2" xyz="-${length_bar} 0 ${length_bar/2}"
     rpy="0 -${pi/2} 0" />
-  <xacro:bar name="layer1" />
+  <xacro:bar name="layer1" length="${length_bar}" width="${width_bar}" thickness="${thickness_bar}" />
   <xacro:fixed_joint parent="map" child="layer1" xyz="-${length_bar/2} 0 ${length_bar}" rpy="0 0 0" />
-  <xacro:bar name="layer2" />
+  <xacro:bar name="layer2" length="${length_bar}" width="${width_bar}" thickness="${thickness_bar}" />
   <xacro:fixed_joint parent="map" child="layer2" xyz="-${length_bar} -${length_bar/2} ${length_bar}"
     rpy="0 0 -${pi/2}" />
-  <xacro:bar name="leg3" />
+  <xacro:bar name="leg3" length="${length_bar}" width="${width_bar}" thickness="${thickness_bar}" />
   <xacro:fixed_joint parent="map" child="leg3" xyz="-${length_bar} -${length_bar} ${length_bar/2}"
     rpy="0 -${pi/2} 0" />
-  <xacro:bar name="layer3" />
+  <xacro:bar name="layer3" length="${length_bar}" width="${width_bar}" thickness="${thickness_bar}" />
   <xacro:fixed_joint parent="map" child="layer3" xyz="0 -${length_bar/2} ${length_bar}"
     rpy="0 0 -${pi/2}" />
-  <xacro:bar name="leg4" />
+  <xacro:bar name="leg4" length="${length_bar}" width="${width_bar}" thickness="${thickness_bar}" />
   <xacro:fixed_joint parent="map" child="leg4" xyz="0 -${length_bar} ${length_bar/2}"
     rpy="0 -${pi/2} 0" />
-  <xacro:bar name="layer4" />
+  <xacro:bar name="layer4" length="${length_bar}" width="${width_bar}" thickness="${thickness_bar}" />
   <xacro:fixed_joint parent="map" child="layer4" xyz="-${length_bar/2} -${length_bar} ${length_bar}"
     rpy="0 0 0" />
-  <xacro:bar name="xaxis" />
+  <xacro:bar name="xaxis" length="${length_bar}" width="${width_bar}" thickness="${thickness_bar}" />
   <xacro:prismatic_joint parent="map" child="xaxis"
     xyz="0 -${length_bar/2} ${length_bar}"
@@ -79,5 +79,5 @@
     lower="-${length_bar}" upper="0" />
   <!-- Make the below small the dimensions of ${width_bar} ${width_bar} ${width_bar} -->
-  <xacro:bar name="yaxis" />
+  <xacro:bar name="yaxis" length="${length_bar}" width="${width_bar}" thickness="${thickness_bar}" />
   <xacro:prismatic_joint parent="xaxis" child="yaxis"
     xyz="${width_bar} 0 0"

Commit message: I changed one error for another

File: workspace/src/gantry2/urdf/gantry.xacro (robot description, xacro)
@@ -93,3 +93,101 @@
     axis="1 0 0"
     lower="-${length_bar/2}" upper="${length_bar/2}" />
+  <ros2_control name="GazeboSimSystem" type="system">
+    <hardware>
+      <plugin>gazebo_ros2_control/GazeboSystem</plugin>
+    </hardware>
+    <joint name="joint_a1">
+      <!--<command_interface
+      name="position"/>-->
+      <command_interface name="position_pid" />
+      <command_interface name="effort" />
+      <state_interface name="position">
+        <param name="initial_value">0.0</param>
+      </state_interface>
+      <state_interface name="velocity" />
+    </joint>
+    <joint name="joint_a2">
+      <!--<command_interface
+      name="position"/>-->
+      <command_interface name="position_pid" />
+      <command_interface name="effort" />
+      <state_interface name="position">
+        <param name="initial_value">0.0</param>
+      </state_interface>
+      <state_interface name="velocity" />
+    </joint>
+    <joint name="joint_a3">
+      <!--<command_interface
+      name="position"/>-->
+      <command_interface name="position_pid" />
+      <command_interface name="effort" />
+      <state_interface name="position">
+        <param name="initial_value">0.0</param>
+      </state_interface>
+      <state_interface name="velocity" />
+    </joint>
+    <sensor name="joint_a1_force_torque">
+      <state_interface name="force.x" />
+      <state_interface name="force.y" />
+      <state_interface name="force.z" />
+      <state_interface name="torque.x" />
+      <state_interface name="torque.y" />
+      <state_interface name="torque.z" />
+    </sensor>
+    <sensor name="joint_a2_force_torque">
+      <state_interface name="force.x" />
+      <state_interface name="force.y" />
+      <state_interface name="force.z" />
+      <state_interface name="torque.x" />
+      <state_interface name="torque.y" />
+      <state_interface name="torque.z" />
+    </sensor>
+    <sensor name="joint_a3_force_torque">
+      <state_interface name="force.x" />
+      <state_interface name="force.y" />
+      <state_interface name="force.z" />
+      <state_interface name="torque.x" />
+      <state_interface name="torque.y" />
+      <state_interface name="torque.z" />
+    </sensor>
+  </ros2_control>
+  <gazebo>
+    <plugin name="gazebo_ros2_control" filename="libgazebo_ros2_control.so">
+      <!-- <parameters>$(find six_dof_arm)/config/six_dof_arm_controllers.yaml</parameters> -->
+      <parameters>$(find gantry2_moveit_config)/config/ros2_controllers.yaml</parameters>
+    </plugin>
+  </gazebo>
+  <gazebo reference="joint_a1">
+    <sensor name="joint_a1_force_torque" type="force_torque">
+      <always_on>true</always_on>
+      <update_rate>100.0</update_rate>
+      <visualize>true</visualize>
+      <force_torque>
+        <frame>sensor</frame>
+        <measure_direction>child_to_parent</measure_direction>
+      </force_torque>
+    </sensor>
+  </gazebo>
+  <gazebo reference="joint_a2">
+    <sensor name="joint_a2_force_torque" type="force_torque">
+      <always_on>true</always_on>
+      <update_rate>100.0</update_rate>
+      <visualize>true</visualize>
+      <force_torque>
+        <frame>sensor</frame>
+        <measure_direction>child_to_parent</measure_direction>
+      </force_torque>
+    </sensor>
+  </gazebo>
+  <gazebo reference="joint_a3">
+    <sensor name="joint_a3_force_torque" type="force_torque">
+      <always_on>true</always_on>
+      <update_rate>100.0</update_rate>
+      <visualize>true</visualize>
+      <force_torque>
+        <frame>sensor</frame>
+        <measure_direction>child_to_parent</measure_direction>
+      </force_torque>
+    </sensor>
+  </gazebo>
 </robot>
