Commit message: Working gantry, need to add end effector

File: workspace/src/gantry2/urdf/gantry.xacro (robot description, xacro)
@@ -97,8 +97,8 @@
       <plugin>gazebo_ros2_control/GazeboSystem</plugin>
     </hardware>
-    <joint name="joint_a1">
+    <joint name="map_to_xaxis">
       <!--<command_interface
       name="position"/>-->
-      <command_interface name="position_pid" />
+      <command_interface name="position" />
       <command_interface name="effort" />
       <state_interface name="position">
@@ -107,8 +107,8 @@
       <state_interface name="velocity" />
     </joint>
-    <joint name="joint_a2">
+    <joint name="xaxis_to_yaxis">
       <!--<command_interface
       name="position"/>-->
-      <command_interface name="position_pid" />
+      <command_interface name="position" />
       <command_interface name="effort" />
       <state_interface name="position">
@@ -117,8 +117,8 @@
       <state_interface name="velocity" />
     </joint>
-    <joint name="joint_a3">
+    <joint name="yaxis_to_zaxis">
       <!--<command_interface
       name="position"/>-->
-      <command_interface name="position_pid" />
+      <command_interface name="position" />
       <command_interface name="effort" />
       <state_interface name="position">
@@ -158,5 +158,5 @@
     </plugin>
   </gazebo>
-  <gazebo reference="joint_a1">
+  <gazebo reference="map_to_xaxis">
     <sensor name="joint_a1_force_torque" type="force_torque">
       <always_on>true</always_on>
@@ -169,5 +169,5 @@
     </sensor>
   </gazebo>
-  <gazebo reference="joint_a2">
+  <gazebo reference="xaxis_to_yaxis">
     <sensor name="joint_a2_force_torque" type="force_torque">
       <always_on>true</always_on>
@@ -180,5 +180,5 @@
     </sensor>
   </gazebo>
-  <gazebo reference="joint_a3">
+  <gazebo reference="yaxis_to_zaxis">
     <sensor name="joint_a3_force_torque" type="force_torque">
       <always_on>true</always_on>

Commit message: Committing before I rebuild everything, I believe a symlink broke

File: workspace/src/gantry2/urdf/gantry.xacro (robot description, xacro)
@@ -93,4 +93,23 @@
     axis="1 0 0"
     lower="-${length_bar/2}" upper="${length_bar/2}" />
+  <link name="eemount">
+    <visual>
+      <geometry>
+        <cylinder length="0.01" radius="0.05" />
+      </geometry>
+    </visual>
+    <collision>
+      <geometry>
+        <cylinder length="0.01" radius="0.05" />
+      </geometry>
+    </collision>
+  </link>
+  <joint name="zaxis_to_eemount" type="revolute">
+    <parent link="zaxis" />
+    <child link="eemount" />
+    <origin xyz="-${length_bar/2 + width_bar} 0 0" rpy="0 ${pi/2} 0" />
+    <axis xyz="0 0 1" />
+    <limit lower="-1.57" upper="1.57" effort="5" velocity="1" />
+  </joint>
   <ros2_control name="GazeboSimSystem" type="system">
     <hardware>
@@ -118,4 +137,14 @@
     </joint>
     <joint name="yaxis_to_zaxis">
+      <!--<command_interface
+      name="position"/>-->
+      <command_interface name="position" />
+      <command_interface name="effort" />
+      <state_interface name="position">
+        <param name="initial_value">0.0</param>
+      </state_interface>
+      <state_interface name="velocity" />
+    </joint>
+    <joint name="zaxis_to_eemount">
       <!--<command_interface
       name="position"/>-->

File: workspace/src/gantry2_moveit_config/config/rectangular_gantry.ros2_control.xacro (robot description, xacro)
@@ -29,4 +29,11 @@
                 <state_interface name="velocity"/>
             </joint>
+            <joint name="zaxis_to_eemount">
+                <command_interface name="position"/>
+                <state_interface name="position">
+                  <param name="initial_value">${initial_positions['zaxis_to_eemount']}</param>
+                </state_interface>
+                <state_interface name="velocity"/>
+            </joint>
         </ros2_control>
     </xacro:macro>

Commit message: Gazebo and rviz status is agreeing, however I need to get the ee_controller to spawn

File: workspace/src/gantry2/urdf/gantry.xacro (robot description, xacro)
@@ -95,4 +95,5 @@
   <link name="eemount">
     <visual>
+      <origin xyz="0 0 0" rpy="0 0 0" />
       <geometry>
         <cylinder length="0.01" radius="0.05" />
@@ -100,8 +101,14 @@
     </visual>
     <collision>
+      <origin xyz="0 0 0" rpy="0 0 0" />
       <geometry>
         <cylinder length="0.01" radius="0.05" />
       </geometry>
     </collision>
+    <inertial>
+      <origin xyz="0 0 0" rpy="0 0 0" />
+      <mass value="${mass_bar}" />
+      <inertia ixx="1.0" ixy="0" ixz="0" iyy="1.0" iyz="0" izz="1.0" />
+    </inertial>
   </link>
   <joint name="zaxis_to_eemount" type="revolute">
@@ -120,5 +127,5 @@
       name="position"/>-->
       <command_interface name="position" />
-      <command_interface name="effort" />
+      <!-- <command_interface name="effort" /> -->
       <state_interface name="position">
         <param name="initial_value">0.0</param>
@@ -130,5 +137,5 @@
       name="position"/>-->
       <command_interface name="position" />
-      <command_interface name="effort" />
+      <!-- <command_interface name="effort" /> -->
       <state_interface name="position">
         <param name="initial_value">0.0</param>
@@ -140,5 +147,5 @@
       name="position"/>-->
       <command_interface name="position" />
-      <command_interface name="effort" />
+      <!-- <command_interface name="effort" /> -->
       <state_interface name="position">
         <param name="initial_value">0.0</param>
@@ -150,5 +157,5 @@
       name="position"/>-->
       <command_interface name="position" />
-      <command_interface name="effort" />
+      <!-- <command_interface name="effort" /> -->
       <state_interface name="position">
         <param name="initial_value">0.0</param>

Commit message: Working

File: workspace/src/gantry2/urdf/gantry.xacro (robot description, xacro)
@@ -119,111 +119,4 @@
     <limit lower="-1.57" upper="1.57" effort="5" velocity="1" />
   </joint>
-  <ros2_control name="GazeboSimSystem" type="system">
-    <hardware>
-      <plugin>gazebo_ros2_control/GazeboSystem</plugin>
-    </hardware>
-    <joint name="map_to_xaxis">
-      <!--<command_interface
-      name="position"/>-->
-      <command_interface name="position" />
-      <!-- <command_interface name="effort" /> -->
-      <state_interface name="position">
-        <param name="initial_value">0.0</param>
-      </state_interface>
-      <state_interface name="velocity" />
-    </joint>
-    <joint name="xaxis_to_yaxis">
-      <!--<command_interface
-      name="position"/>-->
-      <command_interface name="position" />
-      <!-- <command_interface name="effort" /> -->
-      <state_interface name="position">
-        <param name="initial_value">0.0</param>
-      </state_interface>
-      <state_interface name="velocity" />
-    </joint>
-    <joint name="yaxis_to_zaxis">
-      <!--<command_interface
-      name="position"/>-->
-      <command_interface name="position" />
-      <!-- <command_interface name="effort" /> -->
-      <state_interface name="position">
-        <param name="initial_value">0.0</param>
-      </state_interface>
-      <state_interface name="velocity" />
-    </joint>
-    <joint name="zaxis_to_eemount">
-      <!--<command_interface
-      name="position"/>-->
-      <command_interface name="position" />
-      <!-- <command_interface name="effort" /> -->
-      <state_interface name="position">
-        <param name="initial_value">0.0</param>
-      </state_interface>
-      <state_interface name="velocity" />
-    </joint>
-    <sensor name="joint_a1_force_torque">
-      <state_interface name="force.x" />
-      <state_interface name="force.y" />
-      <state_interface name="force.z" />
-      <state_interface name="torque.x" />
-      <state_interface name="torque.y" />
-      <state_interface name="torque.z" />
-    </sensor>
-    <sensor name="joint_a2_force_torque">
-      <state_interface name="force.x" />
-      <state_interface name="force.y" />
-      <state_interface name="force.z" />
-      <state_interface name="torque.x" />
-      <state_interface name="torque.y" />
-      <state_interface name="torque.z" />
-    </sensor>
-    <sensor name="joint_a3_force_torque">
-      <state_interface name="force.x" />
-      <state_interface name="force.y" />
-      <state_interface name="force.z" />
-      <state_interface name="torque.x" />
-      <state_interface name="torque.y" />
-      <state_interface name="torque.z" />
-    </sensor>
-  </ros2_control>
-  <gazebo>
-    <plugin name="gazebo_ros2_control" filename="libgazebo_ros2_control.so">
-      <!-- <parameters>$(find six_dof_arm)/config/six_dof_arm_controllers.yaml</parameters> -->
-      <parameters>$(find gantry2_moveit_config)/config/ros2_controllers.yaml</parameters>
-    </plugin>
-  </gazebo>
-  <gazebo reference="map_to_xaxis">
-    <sensor name="joint_a1_force_torque" type="force_torque">
-      <always_on>true</always_on>
-      <update_rate>100.0</update_rate>
-      <visualize>true</visualize>
-      <force_torque>
-        <frame>sensor</frame>
-        <measure_direction>child_to_parent</measure_direction>
-      </force_torque>
-    </sensor>
-  </gazebo>
-  <gazebo reference="xaxis_to_yaxis">
-    <sensor name="joint_a2_force_torque" type="force_torque">
-      <always_on>true</always_on>
-      <update_rate>100.0</update_rate>
-      <visualize>true</visualize>
-      <force_torque>
-        <frame>sensor</frame>
-        <measure_direction>child_to_parent</measure_direction>
-      </force_torque>
-    </sensor>
-  </gazebo>
-  <gazebo reference="yaxis_to_zaxis">
-    <sensor name="joint_a3_force_torque" type="force_torque">
-      <always_on>true</always_on>
-      <update_rate>100.0</update_rate>
-      <visualize>true</visualize>
-      <force_torque>
-        <frame>sensor</frame>
-        <measure_direction>child_to_parent</measure_direction>
-      </force_torque>
-    </sensor>
-  </gazebo>
+  <xacro:include filename="$(find gantry2)/urdf/ros2_control.xacro" />
 </robot>

Commit message: Breaking apart my xacro

File: workspace/src/gantry2/urdf/gantry.xacro (robot description, xacro)
@@ -1,75 +1,5 @@
 <?xml version="1.0"?>
 <robot xmlns:xacro="http://www.ros.org/wiki/xacro" name="rectangular_gantry">
-  <xacro:property name="length_bar" value="1" />    <!-- travel along X (m) -->
-  <xacro:property name="thickness_bar" value="0.02" />    <!-- travel along X (m) -->
-  <xacro:property name="width_bar" value="0.02" />    <!-- travel along X (m) -->
-  <xacro:property name="mass_bar" value="1" />    <!-- travel along X (m) -->
-  <!-- Macro for a bar -->
-  <xacro:macro name="bar" params="name length width thickness">
-    <link name="${name}">
-      <visual>
-        <origin xyz="0 0 0" rpy="0 0 0" />
-        <geometry>
-          <box size="${length} ${width} ${thickness}" />
-        </geometry>
-        <material name="gray">
-          <color rgba="0.6 0.6 0.6 1.0" />
-        </material>
-      </visual>
-      <collision>
-        <origin xyz="0 0 0" rpy="0 0 0" />
-        <geometry>
-          <box size="${length} ${width} ${thickness}" />
-        </geometry>
-      </collision>
-      <inertial>
-        <origin xyz="0 0 0" rpy="0 0 0" />
-        <mass value="${mass_bar}" />
-        <inertia ixx="1.0" ixy="0" ixz="0" iyy="1.0" iyz="0" izz="1.0" />
-      </inertial>
-    </link>
-  </xacro:macro>
-  <!-- Macro for a fixed joint -->
-  <xacro:macro name="fixed_joint" params="parent child xyz rpy">
-    <joint name="${parent}_to_${child}" type="fixed">
-      <parent link="${parent}" />
-      <child link="${child}" />
-      <origin xyz="${xyz}" rpy="${rpy}" />
-    </joint>
-  </xacro:macro>
-  <xacro:macro name="prismatic_joint" params="parent child xyz rpy axis lower upper">
-    <joint name="${parent}_to_${child}" type="prismatic">
-      <parent link="${parent}" />
-      <child link="${child}" />
-      <origin xyz="${xyz}" rpy="${rpy}" />
-      <axis xyz="${axis}" />
-      <limit lower="${lower}" upper="${upper}" effort="100" velocity="1.0" />
-    </joint>
-  </xacro:macro>
-  <!-- Base link -->
-  <link name="map" />
-  <!-- Bars + joints -->
-  <xacro:bar name="leg1" length="${length_bar}" width="${width_bar}" thickness="${thickness_bar}" />
-  <xacro:fixed_joint parent="map" child="leg1" xyz="0 0 ${length_bar/2}" rpy="0 -${pi/2} 0" />
-  <xacro:bar name="leg2" length="${length_bar}" width="${width_bar}" thickness="${thickness_bar}" />
-  <xacro:fixed_joint parent="map" child="leg2" xyz="-${length_bar} 0 ${length_bar/2}"
-    rpy="0 -${pi/2} 0" />
-  <xacro:bar name="layer1" length="${length_bar}" width="${width_bar}" thickness="${thickness_bar}" />
-  <xacro:fixed_joint parent="map" child="layer1" xyz="-${length_bar/2} 0 ${length_bar}" rpy="0 0 0" />
-  <xacro:bar name="layer2" length="${length_bar}" width="${width_bar}" thickness="${thickness_bar}" />
-  <xacro:fixed_joint parent="map" child="layer2" xyz="-${length_bar} -${length_bar/2} ${length_bar}"
-    rpy="0 0 -${pi/2}" />
-  <xacro:bar name="leg3" length="${length_bar}" width="${width_bar}" thickness="${thickness_bar}" />
-  <xacro:fixed_joint parent="map" child="leg3" xyz="-${length_bar} -${length_bar} ${length_bar/2}"
-    rpy="0 -${pi/2} 0" />
-  <xacro:bar name="layer3" length="${length_bar}" width="${width_bar}" thickness="${thickness_bar}" />
-  <xacro:fixed_joint parent="map" child="layer3" xyz="0 -${length_bar/2} ${length_bar}"
-    rpy="0 0 -${pi/2}" />
-  <xacro:bar name="leg4" length="${length_bar}" width="${width_bar}" thickness="${thickness_bar}" />
-  <xacro:fixed_joint parent="map" child="leg4" xyz="0 -${length_bar} ${length_bar/2}"
-    rpy="0 -${pi/2} 0" />
-  <xacro:bar name="layer4" length="${length_bar}" width="${width_bar}" thickness="${thickness_bar}" />
-  <xacro:fixed_joint parent="map" child="layer4" xyz="-${length_bar/2} -${length_bar} ${length_bar}"
-    rpy="0 0 0" />
+  <xacro:include filename="$(find gantry2)/urdf/bars.xacro" />
   <xacro:bar name="xaxis" length="${length_bar}" width="${width_bar}" thickness="${thickness_bar}" />
   <xacro:prismatic_joint parent="map" child="xaxis"
