Commit message: Broken up completely

File: workspace/src/gantry2/urdf/bars.xacro (robot description, xacro)
@@ -72,3 +72,24 @@
   <xacro:fixed_joint parent="map" child="layer4" xyz="-${length_bar/2} -${length_bar} ${length_bar}"
     rpy="0 0 0" />
+  <xacro:bar name="xaxis" length="${length_bar}" width="${width_bar}" thickness="${thickness_bar}" />
+  <xacro:prismatic_joint parent="map" child="xaxis"
+    xyz="0 -${length_bar/2} ${length_bar + thickness_bar}"
+    rpy="0 0 -${pi/2}"
+    axis="0 1 0"
+    lower="-${length_bar}" upper="0" />
+  <!-- Make the below small the dimensions of ${width_bar} ${width_bar} ${width_bar} -->
+  <xacro:bar name="yaxis" length="${width_bar}" width="${width_bar + width_bar + width_bar}"
+    thickness="${width_bar}" />
+  <xacro:prismatic_joint parent="xaxis" child="yaxis"
+    xyz="-${width_bar + width_bar} -${width_bar} ${thickness_bar}"
+    rpy="0 -${pi/2} 0"
+    axis="0 0 1"
+    lower="-${length_bar/2}" upper="${length_bar/2}" />
+  <xacro:bar name="zaxis" length="${length_bar}" width="${width_bar}"
+    thickness="${thickness_bar}" />
+  <xacro:prismatic_joint parent="yaxis" child="zaxis"
+    xyz="-${width_bar} -${width_bar} ${width_bar}"
+    rpy="0 0 0"
+    axis="1 0 0"
+    lower="-${length_bar/2}" upper="${length_bar/2}" />
 </robot>

File: workspace/src/gantry2/urdf/gantry.xacro (robot description, xacro)
@@ -2,51 +2,5 @@
 <robot xmlns:xacro="http://www.ros.org/wiki/xacro" name="rectangular_gantry">
   <xacro:include filename="$(find gantry2)/urdf/bars.xacro" />
-  <xacro:bar name="xaxis" length="${length_bar}" width="${width_bar}" thickness="${thickness_bar}" />
-  <xacro:prismatic_joint parent="map" child="xaxis"
-    xyz="0 -${length_bar/2} ${length_bar + thickness_bar}"
-    rpy="0 0 -${pi/2}"
-    axis="0 1 0"
-    lower="-${length_bar}" upper="0" />
-  <!-- Make the below small the dimensions of ${width_bar} ${width_bar} ${width_bar} -->
-  <xacro:bar name="yaxis" length="${width_bar}" width="${width_bar + width_bar + width_bar}"
-    thickness="${width_bar}" />
-  <xacro:prismatic_joint parent="xaxis" child="yaxis"
-    xyz="-${width_bar + width_bar} -${width_bar} ${thickness_bar}"
-    rpy="0 -${pi/2} 0"
-    axis="0 0 1"
-    lower="-${length_bar/2}" upper="${length_bar/2}" />
-  <xacro:bar name="zaxis" length="${length_bar}" width="${width_bar}"
-    thickness="${thickness_bar}" />
-  <xacro:prismatic_joint parent="yaxis" child="zaxis"
-    xyz="-${width_bar} -${width_bar} ${width_bar}"
-    rpy="0 0 0"
-    axis="1 0 0"
-    lower="-${length_bar/2}" upper="${length_bar/2}" />
-  <link name="eemount">
-    <visual>
-      <origin xyz="0 0 0" rpy="0 0 0" />
-      <geometry>
-        <cylinder length="0.01" radius="0.05" />
-      </geometry>
-    </visual>
-    <collision>
-      <origin xyz="0 0 0" rpy="0 0 0" />
-      <geometry>
-        <cylinder length="0.01" radius="0.05" />
-      </geometry>
-    </collision>
-    <inertial>
-      <origin xyz="0 0 0" rpy="0 0 0" />
-      <mass value="${mass_bar}" />
-      <inertia ixx="1.0" ixy="0" ixz="0" iyy="1.0" iyz="0" izz="1.0" />
-    </inertial>
-  </link>
-  <joint name="zaxis_to_eemount" type="revolute">
-    <parent link="zaxis" />
-    <child link="eemount" />
-    <origin xyz="-${length_bar/2 + width_bar} 0 0" rpy="0 ${pi/2} 0" />
-    <axis xyz="0 0 1" />
-    <limit lower="-1.57" upper="1.57" effort="5" velocity="1" />
-  </joint>
+  <xacro:include filename="$(find gantry2)/urdf/ee1.xacro" />
   <xacro:include filename="$(find gantry2)/urdf/ros2_control.xacro" />
 </robot>

Commit message: Figured out how to pull wrenches, just need to bolt to the ground

File: workspace/src/gantry2/urdf/bars.xacro (robot description, xacro)
@@ -4,5 +4,5 @@
   <xacro:property name="thickness_bar" value="0.02" />    <!-- travel along X (m) -->
   <xacro:property name="width_bar" value="0.02" />    <!-- travel along X (m) -->
-  <xacro:property name="mass_bar" value="1" />    <!-- travel along X (m) -->
+  <xacro:property name="mass_bar" value="30" />    <!-- weight (kg) -->
   <!-- Macro for a bar -->
   <xacro:macro name="bar" params="name length width thickness">
