Commit message: Working using xacro macros

File: workspace/src/gantry2/urdf/ee3.xacro (robot description, xacro)
@@ -3,5 +3,5 @@
   <!-- Macro: link + joint with configurable parameters -->
   <xacro:macro name="simple_link_with_joint"
-    params="name parent geom_type geom_size
+    params="name parent geom_type geom_size geom_length geom_radius
             link_origin_xyz link_origin_rpy
             joint_type joint_origin_xyz joint_origin_rpy joint_axis
@@ -16,5 +16,5 @@
           </xacro:if>
           <xacro:if value="${geom_type == 'cylinder'}">
-            <cylinder length="${geom_size[0]}" radius="${geom_size[1]}" />
+            <cylinder length="${geom_length}" radius="${geom_radius}" />
           </xacro:if>
         </geometry>
@@ -27,5 +27,5 @@
           </xacro:if>
           <xacro:if value="${geom_type == 'cylinder'}">
-            <cylinder length="${geom_size[0]}" radius="${geom_size[1]}" />
+            <cylinder length="${geom_length}" radius="${geom_radius}" />
           </xacro:if>
         </geometry>
@@ -46,31 +46,25 @@
     </joint>
   </xacro:macro>
-  <link name="eemount">
-    <visual>
-      <origin xyz="0 0 0" rpy="0 0 0" />
-      <geometry>
-        <cylinder length="0.01" radius="0.05" />
-      </geometry>
-    </visual>
-    <collision>
-      <origin xyz="0 0 0" rpy="0 0 0" />
-      <geometry>
-        <cylinder length="0.01" radius="0.05" />
-      </geometry>
-    </collision>
-    <inertial>
-      <origin xyz="0 0 0" rpy="0 0 0" />
-      <mass value="${mass_bar}" />
-      <inertia ixx="1.0" iyy="1.0" izz="1.0" ixy="0" ixz="0" iyz="0" />
-    </inertial>
-  </link>
-  <joint name="zaxis_to_eemount" type="revolute">
-    <parent link="zaxis" />
-    <child link="eemount" />
-    <origin xyz="-${length_bar/2 + width_bar} 0 0" rpy="0 ${pi/2} 0" />
-    <axis xyz="0 0 1" />
-    <limit lower="-1.57" upper="1.57" effort="5" velocity="1" />
-  </joint>
-  <!-- Example usage: left finger -->
+  <!-- EEMount using the macro (cylinder) -->
+  <xacro:simple_link_with_joint
+    name="eemount"
+    parent="zaxis"
+    geom_type="cylinder"
+    geom_size=""
+    geom_length="0.01"
+    geom_radius="0.05"
+    link_origin_xyz="0 0 0"
+    link_origin_rpy="0 0 0"
+    joint_type="revolute"
+    joint_origin_xyz="-${length_bar/2 + width_bar} 0 0"
+    joint_origin_rpy="0 ${pi/2} 0"
+    joint_axis="0 0 1"
+    limit_lower="-1.57"
+    limit_upper="1.57"
+    limit_effort="5"
+    limit_velocity="1"
+    mass="${mass_bar}"
+    ixx="1.0" iyy="1.0" izz="1.0" />
+  <!-- Left finger (box) -->
   <xacro:simple_link_with_joint
     name="left_finger"
@@ -78,4 +72,5 @@
     geom_type="box"
     geom_size="0.02 0.1 0.02"
+    geom_length="0" geom_radius="0"
     link_origin_xyz="0 0.05 0"
     link_origin_rpy="0 0 0"
@@ -90,5 +85,5 @@
     mass="0.05"
     ixx="0.0001" iyy="0.0001" izz="0.0001" />
-  <!-- Example usage: right finger -->
+  <!-- Right finger (box) -->
   <xacro:simple_link_with_joint
     name="right_finger"
@@ -96,4 +91,5 @@
     geom_type="box"
     geom_size="0.02 0.1 0.02"
+    geom_length="0" geom_radius="0"
     link_origin_xyz="0 -0.05 0"
     link_origin_rpy="0 0 0"
