Commit message: Working separation

File: workspace/src/gantry2/urdf/ros2_control.xacro (robot description, xacro)
@@ -6,5 +6,7 @@
       <plugin>gazebo_ros2_control/GazeboSystem</plugin>
     </hardware>
-    <!-- Joints -->
+    <!--
+    ======================================================================================================================================== -->
+    <!-- Gantry part -->
     <joint name="map_to_xaxis">
       <command_interface name="position" />
@@ -28,12 +30,4 @@
       <state_interface name="velocity" />
     </joint>
-    <joint name="zaxis_to_eemount">
-      <command_interface name="position" />
-      <state_interface name="position">
-        <param name="initial_value">0.0</param>
-      </state_interface>
-      <state_interface name="velocity" />
-    </joint>
-    <!-- Force/Torque Sensors -->
     <sensor name="joint_a1_force_torque">
       <state_interface name="force.x" />
@@ -60,6 +54,21 @@
       <state_interface name="torque.z" />
     </sensor>
+    <!--
+    ======================================================================================================================================== -->
+    <!-- Gantry part -->
+    <!--
+    ======================================================================================================================================== -->
+    <!-- End effector part -->
+    <joint name="zaxis_to_eemount">
+      <command_interface name="position" />
+      <state_interface name="position">
+        <param name="initial_value">0.0</param>
+      </state_interface>
+      <state_interface name="velocity" />
+    </joint>
+    <!--
+    ======================================================================================================================================== -->
+    <!-- End effector part -->
   </ros2_control>
-  <!-- Gazebo plugin for ros2_control -->
   <gazebo>
     <plugin name="gazebo_ros2_control" filename="libgazebo_ros2_control.so">
@@ -67,5 +76,7 @@
     </plugin>
   </gazebo>
-  <!-- Gazebo FT Sensors -->
+  <!--
+  ======================================================================================================================================== -->
+  <!-- Gantry part -->
   <gazebo reference="map_to_xaxis">
     <sensor name="joint_a1_force_torque" type="force_torque">
@@ -101,3 +112,6 @@
     </sensor>
   </gazebo>
+  <!--
+  ======================================================================================================================================== -->
+  <!-- Gantry part -->
 </robot>

Commit message: Made some changes to moveit. Am going to move back, however. I will do this new technique without moveit_servo

File: workspace/src/gantry2/urdf/ros2_control.xacro (robot description, xacro)
@@ -11,5 +11,4 @@
     <joint name="map_to_xaxis">
       <command_interface name="position" />
-      <command_interface name="velocity" />
       <state_interface name="position">
         <param name="initial_value">0.0</param>
@@ -19,5 +18,4 @@
     <joint name="xaxis_to_yaxis">
       <command_interface name="position" />
-      <command_interface name="velocity" />
       <state_interface name="position">
         <param name="initial_value">0.0</param>
@@ -27,5 +25,4 @@
     <joint name="yaxis_to_zaxis">
       <command_interface name="position" />
-      <command_interface name="velocity" />
       <state_interface name="position">
         <param name="initial_value">0.0</param>
@@ -65,5 +62,4 @@
     <joint name="zaxis_to_eemount">
       <command_interface name="position" />
-      <command_interface name="velocity" />
       <state_interface name="position">
         <param name="initial_value">0.0</param>
@@ -73,5 +69,4 @@
     <joint name="gripper_left_joint">
       <command_interface name="position" />
-      <command_interface name="velocity" />
       <state_interface name="position">
         <param name="initial_value">0.0</param>
@@ -81,5 +76,4 @@
     <joint name="gripper_right_joint">
       <command_interface name="position" />
-      <command_interface name="velocity" />
       <state_interface name="position">
         <param name="initial_value">0.0</param>

File: workspace/src/gantry2_moveit_config/config/rectangular_gantry.ros2_control.xacro (robot description, xacro)
@@ -43,11 +43,4 @@
                 <state_interface name="velocity"/>
             </joint>
-            <joint name="gripper_right_joint">
-                <command_interface name="position"/>
-                <state_interface name="position">
-                  <param name="initial_value">${initial_positions['gripper_right_joint']}</param>
-                </state_interface>
-                <state_interface name="velocity"/>
-            </joint>
         </ros2_control>
     </xacro:macro>
