Commit message: Basic end effector

File: workspace/src/gantry2/urdf/ee1.xacro (robot description, xacro)
@@ -27,3 +27,58 @@
     <limit lower="-1.57" upper="1.57" effort="5" velocity="1" />
   </joint>
+  <!-- Left finger -->
+  <link name="left_finger">
+    <visual>
+      <origin xyz="0 0.05 0" rpy="0 0 0" />
+      <geometry>
+        <box size="0.02 0.1 0.02" />
+      </geometry>
+      <material name="Gray" />
+    </visual>
+    <collision>
+      <origin xyz="0 0.05 0" rpy="0 0 0" />
+      <geometry>
+        <box size="0.02 0.1 0.02" />
+      </geometry>
+    </collision>
+    <inertial>
+      <mass value="0.05" />
+      <inertia ixx="0.0001" iyy="0.0001" izz="0.0001" ixy="0" ixz="0" iyz="0" />
+    </inertial>
+  </link>
+  <!-- Right finger -->
+  <link name="right_finger">
+    <visual>
+      <origin xyz="0 -0.05 0" rpy="0 0 0" />
+      <geometry>
+        <box size="0.02 0.1 0.02" />
+      </geometry>
+      <material name="Gray" />
+    </visual>
+    <collision>
+      <origin xyz="0 -0.05 0" rpy="0 0 0" />
+      <geometry>
+        <box size="0.02 0.1 0.02" />
+      </geometry>
+    </collision>
+    <inertial>
+      <mass value="0.05" />
+      <inertia ixx="0.0001" iyy="0.0001" izz="0.0001" ixy="0" ixz="0" iyz="0" />
+    </inertial>
+  </link>
+  <joint name="gripper_left_joint" type="prismatic">
+    <parent link="eemount" />
+    <child link="left_finger" />
+    <origin xyz="0 0.05 -0.12" rpy="${pi/2} 0 0" />
+    <axis xyz="0 0 1" /> <!-- slides along +Y -->
+    <limit lower="0.0" upper="0.04" effort="10" velocity="0.1" />
+  </joint>
+  <joint name="gripper_right_joint" type="prismatic">
+    <parent link="eemount" />
+    <child link="right_finger" />
+    <origin xyz="0 -0.05 -0.02" rpy="${pi/2} 0 0" />
+    <axis xyz="0 0 1" /> <!-- slides along -Y -->
+    <limit lower="0.0" upper="0.04" effort="10" velocity="0.1" />
+    <mimic joint="gripper_left_joint" multiplier="-1" offset="0" />
+  </joint>
 </robot>

Commit message: Working perfectly with basic ee, need to integrate with gazebo

File: workspace/src/gantry2/urdf/ee1.xacro (robot description, xacro)
@@ -78,7 +78,7 @@
     <child link="right_finger" />
     <origin xyz="0 -0.05 -0.02" rpy="${pi/2} 0 0" />
-    <axis xyz="0 0 1" /> <!-- slides along -Y -->
+    <axis xyz="0 0 -1" /> <!-- slides along -Y -->
     <limit lower="0.0" upper="0.04" effort="10" velocity="0.1" />
-    <mimic joint="gripper_left_joint" multiplier="-1" offset="0" />
+    <!-- <mimic joint="gripper_left_joint" multiplier="-1" offset="0" /> -->
   </joint>
 </robot>

File: workspace/src/gantry2/urdf/ros2_control.xacro (robot description, xacro)
@@ -67,4 +67,18 @@
       <state_interface name="velocity" />
     </joint>
+    <joint name="gripper_left_joint">
+      <command_interface name="position" />
+      <state_interface name="position">
+        <param name="initial_value">0.0</param>
+      </state_interface>
+      <state_interface name="velocity" />
+    </joint>
+    <joint name="gripper_right_joint">
+      <command_interface name="position" />
+      <state_interface name="position">
+        <param name="initial_value">0.0</param>
+      </state_interface>
+      <state_interface name="velocity" />
+    </joint>
     <!--
     ======================================================================================================================================== -->

Commit message: Working end effector

File: workspace/src/gantry2/urdf/ee1.xacro (robot description, xacro)
@@ -34,5 +34,4 @@
         <box size="0.02 0.1 0.02" />
       </geometry>
-      <material name="Gray" />
     </visual>
     <collision>
@@ -54,5 +53,4 @@
         <box size="0.02 0.1 0.02" />
       </geometry>
-      <material name="Gray" />
     </visual>
     <collision>

File: workspace/src/gantry2_moveit_config/config/rectangular_gantry.ros2_control.xacro (robot description, xacro)
@@ -36,4 +36,18 @@
                 <state_interface name="velocity"/>
             </joint>
+            <joint name="gripper_left_joint">
+                <command_interface name="position"/>
+                <state_interface name="position">
+                  <param name="initial_value">${initial_positions['gripper_left_joint']}</param>
+                </state_interface>
+                <state_interface name="velocity"/>
+            </joint>
+            <joint name="gripper_right_joint">
+                <command_interface name="position"/>
+                <state_interface name="position">
+                  <param name="initial_value">${initial_positions['gripper_right_joint']}</param>
+                </state_interface>
+                <state_interface name="velocity"/>
+            </joint>
         </ros2_control>
     </xacro:macro>

Commit message: Grasping works now, thanks to IFRA_LinkAttacher repo!

File: workspace/src/gantry2/urdf/ee1.xacro (robot description, xacro)
@@ -65,18 +65,20 @@
     </inertial>
   </link>
+  <!-- Left prismatic joint -->
   <joint name="gripper_left_joint" type="prismatic">
     <parent link="eemount" />
     <child link="left_finger" />
     <origin xyz="0 0.05 -0.12" rpy="${pi/2} 0 0" />
-    <axis xyz="0 0 1" /> <!-- slides along +Y -->
-    <limit lower="0.0" upper="0.04" effort="10" velocity="0.1" />
+    <axis xyz="0 0 -1" /> <!-- slides along +Y -->
+    <limit lower="0.0" upper="0.08" effort="10" velocity="0.1" />
   </joint>
+  <!-- Right prismatic joint (mimics left) -->
   <joint name="gripper_right_joint" type="prismatic">
     <parent link="eemount" />
     <child link="right_finger" />
     <origin xyz="0 -0.05 -0.02" rpy="${pi/2} 0 0" />
-    <axis xyz="0 0 -1" /> <!-- slides along -Y -->
-    <limit lower="0.0" upper="0.04" effort="10" velocity="0.1" />
-    <!-- <mimic joint="gripper_left_joint" multiplier="-1" offset="0" /> -->
+    <axis xyz="0 0 1" /> <!-- slides along -Y -->
+    <limit lower="0.0" upper="0.08" effort="10" velocity="0.1" />
+    <mimic joint="gripper_left_joint" multiplier="1" offset="0" />
   </joint>
 </robot>

Commit message: Working

File: workspace/src/gantry2/urdf/ee1.xacro (robot description, xacro)
@@ -25,5 +25,5 @@
     <origin xyz="-${length_bar/2 + width_bar} 0 0" rpy="0 ${pi/2} 0" />
     <axis xyz="0 0 1" />
-    <limit lower="-1.57" upper="1.57" effort="5" velocity="1" />
+    <limit lower="-3.57" upper="3.57" effort="5" velocity="1" />
   </joint>
   <!-- Left finger -->
